Commit message: good

File: src/kinova-ros/kinova_description/urdf/j2s7s300_standalone.xacro (robot description, xacro)
@@ -17,7 +17,7 @@
   <xacro:include filename="$(find kinova_description)/urdf/j2s7s300.xacro" />
   <!-- <xacro:include filename="$(find kinova_description)/urdf/realsense_d435.urdf.xacro" /> -->
-  <link name="root" />
   <!-- for gazebo -->
   <link name="world" />
+  <link name="root" />
   <joint name="connect_root_and_world" type="fixed">
     <child link="root" />
